Commit message: BlueROV2 urdf working, beginning components.xacro

File: orca_description/urdf/bluerov2.urdf.xacro (robot description, xacro)
@@ -1,11 +1,146 @@
-<?xml version="1.0" encoding="UTF-8"?>
+<?xml version="1.0"?>
 <robot name="BlueROV2" xmlns:xacro="http://ros.org/wiki/xacro">
-    <xacro:property name="gazebo_sim" value="True"/>
-    <xacro:include filename="$(find-pkg-share orca_description)/urdf/bluerov2_base.xacro"/>
-    <xacro:bluerov2_base
-        robot_namespace="${namespace}"
-        mass="${mass}">
+    <!--Macro Properties ROV-->
+    <xacro:property name="namespace" value="bluerov2"/>
+    <xacro:property name="mass" value="1"/>
+    <xacro:property name="gz_sim" value="True"/>
+    <!--Sistema de Medição 2-->
+    <xacro:property name="use_sm2" value="True"/>
+    <xacro:property name="sm2_h_res" value="1600"/>
+    <xacro:property name="sm2_v_res" value="1200"/>
+    <xacro:property name="sm2_h_fov" value="1.6757"/> <!--FoV H: 96 deg-->
+    <!--Includes-->
+    <xacro:include filename="bluerov2_base.xacro"/>
+    <xacro:include filename="components.xacro" />
+    <xacro:bluerov2_base robot_namespace="${namespace}"
+                         mass="${mass}"
+                         filename="package://orca_description/models/orca4/meshes/bluerov2.dae"
+        use_gz="${gz_sim}">
     </xacro:bluerov2_base>
-    <xacro:if value="${gazebo_sim}">
-    </xacro:if>
+    <xacro:thruster robot_namespace="${namespace}" motor_n="1"
+                    use_gz="${gz_sim}"
+                    visual_rpy="${pi/2} 0 0"
+                    color="Blue"
+                    axis="0 0 -1"
+                    xyz="0.14 -0.092 0"
+                    rpy="-${pi/2} ${pi/2} ${pi/4}"
+                    uri_mesh="package://orca_description/models/orca4/meshes/t200-cw-prop.dae">
+    </xacro:thruster>
+    <xacro:thruster robot_namespace="${namespace}" motor_n="2"
+                    use_gz="${gz_sim}"
+                    color="Red"
+                    visual_rpy="-${pi/2} 0 0"
+                    axis="0 0 -1"
+                    xyz="0.14 0.092 0"
+                    rpy="-${pi/2} ${pi/2} ${3*pi/4}"
+                    uri_mesh="package://orca_description/models/orca4/meshes/t200-ccw-prop.dae">
+    </xacro:thruster>
+    <xacro:thruster robot_namespace="${namespace}" motor_n="3"
+                    use_gz="${gz_sim}"
+                    color="Red"
+                    visual_rpy="-${pi/2} 0 0"
+                    axis="0 0 -1"
+                    xyz="-0.14 -0.092 0"
+                    rpy="-${pi/2} ${pi/2} ${pi/4}"
+                    uri_mesh="package://orca_description/models/orca4/meshes/t200-ccw-prop.dae">
+    </xacro:thruster>
+    <xacro:thruster robot_namespace="${namespace}" motor_n="4"
+                    use_gz="${gz_sim}"
+                    color="Blue"
+                    visual_rpy="${pi/2} 0 0"
+                    axis="0 0 -1"
+                    xyz="-0.14 0.092 0"
+                    rpy="-${pi/2} ${pi/2} ${3*pi/4}"
+                    uri_mesh="package://orca_description/models/orca4/meshes/t200-cw-prop.dae">
+    </xacro:thruster>
+    <xacro:thruster robot_namespace="${namespace}" motor_n="5"
+                    use_gz="${gz_sim}"
+                    color="Red"
+                    visual_rpy="-${pi/2} 0 ${pi/2}"
+                    axis="0 0 -1"
+                    xyz="0 -0.109 0.077"
+                    rpy="0 0 0"
+                    uri_mesh="package://orca_description/models/orca4/meshes/t200-ccw-prop.dae">
+    </xacro:thruster>
+    <xacro:thruster robot_namespace="${namespace}" motor_n="6"
+                    use_gz="${gz_sim}"
+                    color="Blue"
+                    visual_rpy="${pi/2} 0 ${pi/2}"
+                    axis="0 0 -1"
+                    xyz="0 0.109 0.077"
+                    rpy="0 0 0"
+                    uri_mesh="package://orca_description/models/orca4/meshes/t200-cw-prop.dae">
+    </xacro:thruster>
+    <gazebo>
+        <plugin name="ArduPilotPlugin" filename="libArduPilotPlugin.so">
+            <!-- Port settings -->
+            <fdm_addr>127.0.0.1</fdm_addr>
+            <fdm_port_in>9002</fdm_port_in>
+            <connectionTimeoutMaxCount>5</connectionTimeoutMaxCount>
+            <lock_step>1</lock_step>
+            <!-- Transform from the Gazebo body frame (x-forward, y-left, z-up)
+                 to the ArduPilot body frame (x-forward, y-right, z-down) -->
+            <modelXYZToAirplaneXForwardZDown>0 0 0 ${pi} 0 0</modelXYZToAirplaneXForwardZDown>
+            <!-- Transform from the Gazebo world frame (ENU)
+                 to the ArduPilot world frame (NED) -->
+            <gazeboXYZToNED>0 0 0 ${pi} 0 ${pi/2}</gazeboXYZToNED>
+            <!-- Sensors -->
+            <imuName>imu_sensor</imuName>
+            <!-- Thrusters -->
+            <control channel="0">
+                <jointName>${namespace}/thruster1_joint</jointName>
+                <servo_min>1100</servo_min>
+                <servo_max>1900</servo_max>
+                <type>COMMAND</type>
+                <cmd_topic>/model/orca4/joint/thruster1_joint/cmd_thrust</cmd_topic>
+                <offset>-0.5</offset>
+                <multiplier>100</multiplier>
+            </control>
+            <control channel="1">
+                <jointName>${namespace}/thruster2_joint</jointName>
+                <servo_min>1100</servo_min>
+                <servo_max>1900</servo_max>
+                <type>COMMAND</type>
+                <cmd_topic>/model/orca4/joint/thruster2_joint/cmd_thrust</cmd_topic>
+                <offset>-0.5</offset>
+                <multiplier>100</multiplier>
+            </control>
+            <control channel="2">
+                <jointName>${namespace}/thruster3_joint</jointName>
+                <servo_min>1100</servo_min>
+                <servo_max>1900</servo_max>
+                <type>COMMAND</type>
+                <cmd_topic>/model/orca4/joint/thruster3_joint/cmd_thrust</cmd_topic>
+                <offset>-0.5</offset>
+                <multiplier>100</multiplier>
+            </control>
+            <control channel="3">
+                <jointName>${namespace}/thruster4_joint</jointName>
+                <servo_min>1100</servo_min>
+                <servo_max>1900</servo_max>
+                <type>COMMAND</type>
+                <cmd_topic>/model/orca4/joint/thruster4_joint/cmd_thrust</cmd_topic>
+                <offset>-0.5</offset>
+                <multiplier>100</multiplier>
+            </control>
+            <control channel="4">
+                <jointName>${namespace}/thruster5_joint</jointName>
+                <servo_min>1100</servo_min>
+                <servo_max>1900</servo_max>
+                <type>COMMAND</type>
+                <cmd_topic>/model/orca4/joint/thruster5_joint/cmd_thrust</cmd_topic>
+                <offset>-0.5</offset>
+                <multiplier>100</multiplier>
+            </control>
+            <control channel="5">
+                <jointName>${namespace}/thruster6_joint</jointName>
+                <servo_min>1100</servo_min>
+                <servo_max>1900</servo_max>
+                <type>COMMAND</type>
+                <cmd_topic>/model/orca4/joint/thruster6_joint/cmd_thrust</cmd_topic>
+                <offset>-0.5</offset>
+                <multiplier>100</multiplier>
+            </control>
+        </plugin>
+    </gazebo>
 </robot>

File: orca_description/urdf/bluerov2_base.xacro (robot description, xacro)
@@ -2,17 +2,11 @@
 <robot xmlns:xacro="http://ros.org/wiki/xacro">
     <xacro:macro name="bluerov2_base"
-                 params="robot_namespace mass">
-        <link name="${robot_namespace}/base_link">
-            <inertial>
-                <mass value="${mass}"/>  <!-- [kg] -->
-                <origin xyz="0 0 0"/>
-                <!--                <inertia ixx="0.0" ixy="0.0" ixz="0.0" iyy="0.00" iyz="0.0" izz="0.0"/>-->
-                <xacro:insert_block name="inertia"/>
-            </inertial>
+                 params="robot_namespace mass use_gz filename">
+        <link name="${namespace}/base_link">
             <visual>
                 <origin xyz="0 0 0" rpy="0 0 0"/>
                 <geometry>
-                    <mesh filename="package://orca_description/models/orca4/meshes/bluerov2.dae"
-                          scale="0.25 0.25 0.25"/>
+                    <mesh filename="${filename}"
+                          scale="0.025 0.025 0.025"/>
                 </geometry>
             </visual>
@@ -20,19 +14,22 @@
                 <origin xyz="0 0 0" rpy="0 0 0"/>
                 <geometry>
-                    <box size="0.457 0.338 0.06506286173008947"/>  <!-- [m] [m] [m] -->
+                    <box size="0.4571 0.3381 0.2539"/>  <!-- [m] [m] [m] -->
                 </geometry>
             </collision>
+            <xacro:if value="${use_gz}">
+            <!-- IMU sensor gyro and accel data will be sent to ArduSub -->
+            <sensor name="imu_sensor" type="imu">
+                <!-- Transform from the Gazebo body frame (x-forward, y-left, z-up)
+                     to the ArduPilot body frame (x-forward, y-right, z-down) -->
+                <pose>0 0 0 ${pi} 0 0</pose>
+                <always_on>1</always_on>
+                <update_rate>1000.0</update_rate>
+            </sensor>
+            </xacro:if>
         </link>
-        <!--        <joint name="${robot_namespace}/base_joint" type="fixed">-->
-        <!--            <origin xyz="0 0 0" rpy="0 0 0"/>-->
-        <!--            <parent name="${robot_namespace}/base_link"/>-->
-        <!--            <child name="base_link_visual"/>-->
-        <!--        </joint>-->
-        <!--        <link name="base_link_visual">-->
-        <!--            -->
-        <!--        </link>-->
+        <xacro:if value="${use_gz}">
         <gazebo reference="${robot_namespace}/base_link">
             <plugin filename="gz-sim-hydrodynamics-system" name="gz::sim::systems::Hydrodynamics">
-                <link_name>base_link</link_name>
+                <link_name>${robot_namespace}/base_link</link_name>
                 <water_density>1000</water_density>
                 <!-- Added mass: -->
@@ -59,12 +56,41 @@
             </plugin>
         </gazebo>
+        </xacro:if>
     </xacro:macro>
-    <xacro:macro name="thruster" params="robot_namespace parent motor_n axis xyz rpy">
-        <joint name="${robot_namespace}/thruster${motor_n}_joint" type="revolute">
+    <xacro:macro name="thruster" params="robot_namespace visual_rpy color motor_n axis xyz rpy uri_mesh use_gz">
+        <link name="${namespace}/thruster${motor_n}_link">
+            <visual name="thruster_prop_visual">
+                <origin xyz="0 0 0" rpy="${visual_rpy}"/>
+                <geometry>
+                    <mesh filename="${uri_mesh}"/>
+                </geometry>
+            </visual>
+            <inertial>
+                <mass value="0.002"/>
+                <inertia ixx="1e-3" ixy="0.0" ixz="0.0" iyy="1e-3" iyz="0.0" izz="1e-3"/>
+            </inertial>
+        </link>
+        <joint name="${namespace}/thruster${motor_n}_joint" type="continuous">
+            <parent link="${namespace}/base_link"/>
+            <child link="${namespace}/thruster${motor_n}_link"/>
             <origin xyz="${xyz}" rpy="${rpy}"/>
-            <parent name="${parent}"/>
-            <child name="${robot_namespace}/thruster${motor_n}_link"/>
-            <axis xyz="0 0 -1"/>
+            <axis xyz="${axis}"/>
         </joint>
+        <xacro:if value="${use_gz}">
+            <gazebo>
+                <plugin filename="gz-sim-thruster-system" name="gz::sim::systems::Thruster">
+                    <namespace>${namespace}</namespace>
+                    <joint_name>${namespace}/thruster${motor_n}_joint</joint_name>
+                    <thrust_coefficient>0.02</thrust_coefficient>
+                    <fluid_density>1000</fluid_density>
+                    <propeller_diameter>0.1</propeller_diameter>
+                    <velocity_control>true</velocity_control>
+                    <use_angvel_cmd>False</use_angvel_cmd>
+                </plugin>
+            </gazebo>
+            <gazebo reference="${namespace}/thruster${motor_n}_link">
+                <material>Gazebo/${color}</material>
+            </gazebo>
+        </xacro:if>
     </xacro:macro>
 </robot>
