Commit message: bluerov2 heavy urdf initiate but docker is failing to build

File: orca_description/urdf/bluerov2_base.xacro (robot description, xacro)
@@ -1,6 +1,11 @@
 <?xml version="1.0"?>
 <robot xmlns:xacro="http://ros.org/wiki/xacro">
+    <xacro:macro name="box_inertia" params="x y z mass">
+        <inertia ixx="${0.0833333 * mass * (y*y + z*z)}" ixy="0.0" ixz="0.0"
+                 iyy="${0.0833333 * mass * (x*x + z*z)}" iyz="0.0"
+                 izz="${0.0833333 * mass * (x*x + y*y)}"/>
+    </xacro:macro>
     <xacro:macro name="bluerov2_base"
-                 params="robot_namespace mass use_gz filename">
+                 params="robot_namespace mass use_gz filename x y z heavy">
         <link name="${namespace}/base_link">
             <visual>
@@ -14,7 +19,12 @@
                 <origin xyz="0 0 0" rpy="0 0 0"/>
                 <geometry>
-                    <box size="0.4571 0.3381 0.2539"/>  <!-- [m] [m] [m] -->
+                    <box size="${x} ${y} ${z}"/>  <!-- [m] [m] [m] -->
                 </geometry>
             </collision>
+            <inertial>
+                <mass value="${mass}"/>
+                <origin xyz="0 0 0"/>
+                <xacro:box_inertia mass="${mass}" x="${x}" y="${y}" z="${z}"/>
+=            </inertial>
             <xacro:if value="${use_gz}">
             <!-- IMU sensor gyro and accel data will be sent to ArduSub -->
@@ -48,7 +58,14 @@
                 <nR>0</nR>
                 <!-- Second order stability derivative: -->
-                <xUabsU>-33.800000000000004</xUabsU>
-                <yVabsV>-54.26875</yVabsV>
-                <zWabsW>-73.37135</zWabsW>
+                <xacro:if value="${heavy}">
+                    <xUabsU>-58.42</xUabsU>
+                    <yVabsV>-55.137</yVabsV>
+                    <zWabsW>-124.818</zWabsW>
+                </xacro:if>
+                <xacro:unless value="${heavy}">
+                    <xUabsU>-33.800000000000004</xUabsU>
+                    <yVabsV>-54.26875</yVabsV>
+                    <zWabsW>-73.37135</zWabsW>
+                </xacro:unless>
                 <kPabsP>-4.0</kPabsP>
                 <mQabsQ>-4.0</mQabsQ>

File: orca_description/urdf/bluerov2_heavy.urdf.xacro (robot description, xacro)
@@ -2,6 +2,6 @@
 <robot name="BlueROV2" xmlns:xacro="http://ros.org/wiki/xacro">
     <!--Macro Properties ROV-->
-    <xacro:property name="namespace" value="bluerov2"/>
-    <xacro:property name="mass" value="1"/>
+    <xacro:property name="namespace" value="bluerov2_voris"/>
+    <xacro:property name="mass" value="13"/>
     <xacro:property name="gz_sim" value="True"/>
     <!--Sistema de Medição 2-->
@@ -18,16 +18,16 @@
                          use_gz="${gz_sim}"
                          x="0.457"
-                         y="0.338"
-                         z="0.065"
-                         heavy="False">
+                         y="0.575"
+                         z="0.05"
+                        heavy="True">
     </xacro:bluerov2_base>
     <xacro:thruster robot_namespace="${namespace}" motor_n="1"
                     use_gz="${gz_sim}"
-                    visual_rpy="${pi/2} 0 0"
-                    color="Blue"
-                    axis="0 0 -1"
-                    xyz="0.14 -0.092 0"
-                    rpy="-${pi/2} ${pi/2} ${pi/4}"
-                    uri_mesh="package://orca_description/models/orca4/meshes/t200-cw-prop.dae">
+                    visual_rpy="-${pi/2} 0 0"
+                    color="Blue"
+                    axis="0 0 -1"
+                    xyz="0.14 -0.092 0.0"
+                    rpy="-${pi/2} ${pi/2} -${pi/4}"
+                    uri_mesh="package://orca_description/models/orca4/meshes/t200-ccw-prop.dae">
     </xacro:thruster>
     <xacro:thruster robot_namespace="${namespace}" motor_n="2"
@@ -36,6 +36,6 @@
                     visual_rpy="-${pi/2} 0 0"
                     axis="0 0 -1"
-                    xyz="0.14 0.092 0"
-                    rpy="-${pi/2} ${pi/2} ${3*pi/4}"
+                    xyz="0.14 0.092 0.0"
+                    rpy="-${pi/2} ${pi/2} -${3*pi/4}"
                     uri_mesh="package://orca_description/models/orca4/meshes/t200-ccw-prop.dae">
     </xacro:thruster>
@@ -43,9 +43,9 @@
                     use_gz="${gz_sim}"
                     color="Red"
-                    visual_rpy="-${pi/2} 0 0"
-                    axis="0 0 -1"
-                    xyz="-0.14 -0.092 0"
+                    visual_rpy="${pi/2} 0 0"
+                    axis="0 0 -1"
+                    xyz="-0.15 -0.092 0.0"
                     rpy="-${pi/2} ${pi/2} ${pi/4}"
-                    uri_mesh="package://orca_description/models/orca4/meshes/t200-ccw-prop.dae">
+                    uri_mesh="package://orca_description/models/orca4/meshes/t200-cw-prop.dae">
     </xacro:thruster>
     <xacro:thruster robot_namespace="${namespace}" motor_n="4"
@@ -54,6 +54,6 @@
                     visual_rpy="${pi/2} 0 0"
                     axis="0 0 -1"
-                    xyz="-0.14 0.092 0"
-                    rpy="-${pi/2} ${pi/2} ${3*pi/4}"
+                    xyz="-0.15 0.092 0.0"
+                    rpy="-${pi/2} -${pi/2} ${3*pi/4}"
                     uri_mesh="package://orca_description/models/orca4/meshes/t200-cw-prop.dae">
     </xacro:thruster>
@@ -63,5 +63,5 @@
                     visual_rpy="-${pi/2} 0 ${pi/2}"
                     axis="0 0 -1"
-                    xyz="0 -0.109 0.077"
+                    xyz="0.118 -0.215 0.064"
                     rpy="0 0 0"
                     uri_mesh="package://orca_description/models/orca4/meshes/t200-ccw-prop.dae">
@@ -72,27 +72,45 @@
                     visual_rpy="${pi/2} 0 ${pi/2}"
                     axis="0 0 -1"
-                    xyz="0 0.109 0.077"
-                    rpy="0 0 0"
-                    uri_mesh="package://orca_description/models/orca4/meshes/t200-cw-prop.dae">
-    </xacro:thruster>
-    <xacro:sm2 namespace="${namespace}"
-               camera_name="stereo"
-               parent_link="${namespace}/base_link"
-               frame_rate="60"
-               horizontal_fov="${pi/180*91}"
-               image_width="1600"
-               image_height="1200"
-               image_format="Mono8"
-               min_distance="2"
-               max_distance="10"
-               noise_mean="0.0"
-               noise_stddev="0"
-               enable_visual="1"
-               origin_offset_x="0.055"
-               baseline_y="1"
-               origin_offset_z="-0.001"
-               mass="0.01"
-    >
-    </xacro:sm2>
+                    xyz="0.118 0.215 0.064"
+                    rpy="0 0 0"
+                    uri_mesh="package://orca_description/models/orca4/meshes/t200-cw-prop.dae">
+    </xacro:thruster>
+    <xacro:thruster robot_namespace="${namespace}" motor_n="7"
+                    use_gz="${gz_sim}"
+                    color="Blue"
+                    visual_rpy="${pi/2} 0 ${pi/2}"
+                    axis="0 0 -1"
+                    xyz="-0.118 -0.215 0.064"
+                    rpy="0 0 0"
+                    uri_mesh="package://orca_description/models/orca4/meshes/t200-cw-prop.dae">
+    </xacro:thruster>
+    <xacro:thruster robot_namespace="${namespace}" motor_n="8"
+                    use_gz="${gz_sim}"
+                    color="Blue"
+                    visual_rpy="-${pi/2} 0 ${pi/2}"
+                    axis="0 0 -1"
+                    xyz="-0.118 0.215 0.064"
+                    rpy="0 0 0"
+                    uri_mesh="package://orca_description/models/orca4/meshes/t200-ccw-prop.dae">
+    </xacro:thruster>
+<!--    <xacro:sm2 namespace="${namespace}"-->
+<!--               camera_name="stereo"-->
+<!--               parent_link="${namespace}/base_link"-->
+<!--               frame_rate="60"-->
+<!--               horizontal_fov="${pi/180*91}"-->
+<!--               image_width="1600"-->
+<!--               image_height="1200"-->
+<!--               image_format="Mono8"-->
+<!--               min_distance="2"-->
+<!--               max_distance="10"-->
+<!--               noise_mean="0.0"-->
+<!--               noise_stddev="0"-->
+<!--               enable_visual="1"-->
+<!--               origin_offset_x="0.055"-->
+<!--               baseline_y="1"-->
+<!--               origin_offset_z="-0.001"-->
+<!--               mass="0.01"-->
+<!--    >-->
+<!--    </xacro:sm2>-->
     <xacro:if value="${gz_sim}">
         <gazebo>
@@ -165,4 +183,21 @@
                     <offset>-0.5</offset>
                     <multiplier>100</multiplier>
+                <control channel="6">
+                    <jointName>${namespace}/thruster7_joint</jointName>
+                    <servo_min>1100</servo_min>
+                    <servo_max>1900</servo_max>
+                    <type>COMMAND</type>
+                    <cmd_topic>/model/bluerov2_heavy/joint/thruster7_joint/cmd_thrust</cmd_topic>
+                    <offset>-0.5</offset>
+                    <multiplier>100</multiplier>
+                </control>
+                <control channel="7">
+                    <jointName>${namespace}/thruster8_joint</jointName>
+                    <servo_min>1100</servo_min>
+                    <servo_max>1900</servo_max>
+                    <type>COMMAND</type>
+                    <cmd_topic>/model/bluerov2_heavy/joint/thruster8_joint/cmd_thrust</cmd_topic>
+                    <offset>-0.5</offset>
+                    <multiplier>100</multiplier>
                 </control>
             </plugin>

File: orca_description/urdf/components.xacro (robot description, xacro)
@@ -6,7 +6,7 @@
       baseline_y origin_offset_z mass">
         <joint name="base_to_camera" type="fixed">
-            <parent link="${namespace}/base_link"/>
+            <parent link="${parent_link}"/>
             <child lin="${namespace}/sm2/camera_left_link"/>
-            <origin xyz="${xyz_left}" rpy="${rpy_left}"/>
+            <origin xyz="${origin_offset_x} 0 ${origin_offset_z}" rpy="0 0 0"/>
         </joint>
         <link name="${namespace}/sm2/camera_base_link">
@@ -20,5 +20,5 @@
                 <origin xyz="0 0 0" rpy="${pi/2} 0 ${pi/2}"/>
                 <geometry>
-                    <mesh filename="$(find vant3d_description)/meshes/stereo.dae" scale="1 1 1"/>
+                    <cylinder radius=".015" length="${baseline_y}"/>
                 </geometry>
             </visual>
@@ -36,12 +36,18 @@
         <link name="${namespace}/sm2/camera_left_link">
         </link>
-        <!-- Both cameras in the pair are anchored off the left camera frame. -->
-        <gazebo reference="${namespace}/sm2/camera_left_link">
-            <sensor type="multicamera" name="${namespace}_sm2_stereo_camera">
+        <joint name="${namespace}/camera_right_joint" type="fixed">
+            <origin xyz="${origin_offset_x} -${baseline_y/2} ${origin_offset_z}" rpy="0 0 0"/>
+            <parent link="${namespace}/sm2/camera_base_link"/>
+            <child link="${namespace}/sm2/camera_right_link"/>
+        </joint>
+        <link name="${namespace}/sm2/camera_right_link">
+        </link>
+        <gazebo reference="${namespace}/sm2/camera_right_link">
+            <sensor type="camera" name="${namespace}_sm2_right_camera">
                 <update_rate>${frame_rate}</update_rate>
                 <visualize>false</visualize>
                 <!-- Here we set up the individual cameras of the stereo.yaml head. -->
-                <camera name="left">
-                    <pose>0 0 0 0 0 -0.07</pose>
+                <camera name="right">
+                    <pose>0 0 0 0 0 0</pose>
                     <horizontal_fov>${horizontal_fov}</horizontal_fov>
                     <image>
@@ -63,8 +69,14 @@
                     </noise>
                 </camera>
-                <camera name="right">
-                    <pose>0 ${-baseline_y} 0 0 0 +0.07</pose>
+            </sensor>
+        </gazebo>
+        <gazebo reference="${namespace}/sm2/camera_left_link">
+            <sensor type="camera" name="${namespace}_sm2_left_camera">
+                <update_rate>${frame_rate}</update_rate>
+                <visualize>false</visualize>
+                <!-- Here we set up the individual cameras of the stereo.yaml head. -->
+                <camera name="left">
+                    <pose>0 0 0 0 0 0</pose>
                     <horizontal_fov>${horizontal_fov}</horizontal_fov>
-                    <visualize>false</visualize>
                     <image>
                         <width>${image_width}</width>
@@ -85,19 +97,4 @@
                     </noise>
                 </camera>
-                <!-- Stereo controller, setting the transforms between the two cameras. -->
-                <plugin name="${namespace}_stereo_camera_controller" filename="libgazebo_ros_multicamera.so">
-                    <alwaysOn>true</alwaysOn>
-                    <updateRate>0.0</updateRate>
-                    <cameraName>${camera_name}</cameraName>
-                    <imageTopicName>image_raw</imageTopicName>
-                    <cameraInfoTopicName>camera_info</cameraInfoTopicName>
-                    <frameName>camera_left_link</frameName>
-                    <hackBaseline>${baseline_y}</hackBaseline>
-                    <distortionK1>0.0</distortionK1>
-                    <distortionK2>0.0</distortionK2>
-                    <distortionK3>0.0</distortionK3>
-                    <distortionT1>0.0</distortionT1>
-                    <distortionT2>0.0</distortionT2>
-                </plugin>
             </sensor>
         </gazebo>
